Commit message: Integrate ros2_control and enable differential drive in Gazebo

File: src/forkkun_description/urdf/Forkkun.xacro (robot description, xacro)
@@ -1,7 +1,8 @@
 <?xml version="1.0" ?>
 <robot name="Forkkun" xmlns:xacro="http://www.ros.org/wiki/xacro">
-<xacro:include filename="$(find Forkkun_description)/urdf/materials.xacro" />
-<xacro:include filename="$(find Forkkun_description)/urdf/Forkkun.trans" />
-<xacro:include filename="$(find Forkkun_description)/urdf/Forkkun.gazebo" />
+<xacro:include filename="$(find forkkun_description)/urdf/materials.xacro" />
+<xacro:include filename="$(find forkkun_description)/urdf/Forkkun.trans" />
+<xacro:include filename="$(find forkkun_description)/urdf/Forkkun.gazebo" />
+<xacro:include filename="$(find forkkun_description)/urdf/Forkkun.ros2_control.xacro" />
 <link name="base_link">
   <inertial>
@@ -13,5 +14,5 @@
     <origin xyz="0 0 0" rpy="0 0 0"/>
     <geometry>
-      <mesh filename="file://$(find Forkkun_description)/meshes/base_link.stl" scale="0.001 0.001 0.001"/>
+      <mesh filename="file://$(find forkkun_description)/meshes/base_link.stl" scale="0.001 0.001 0.001"/>
     </geometry>
     <material name="silver"/>
@@ -20,5 +21,5 @@
     <origin xyz="0 0 0" rpy="0 0 0"/>
     <geometry>
-      <mesh filename="file://$(find Forkkun_description)/meshes/base_link.stl" scale="0.001 0.001 0.001"/>
+      <mesh filename="file://$(find forkkun_description)/meshes/base_link.stl" scale="0.001 0.001 0.001"/>
     </geometry>
   </collision>
@@ -33,5 +34,5 @@
     <origin xyz="0.075 0.3 0.36" rpy="0 0 0"/>
     <geometry>
-      <mesh filename="file://$(find Forkkun_description)/meshes/right_wheel_1.stl" scale="0.001 0.001 0.001"/>
+      <mesh filename="file://$(find forkkun_description)/meshes/right_wheel_1.stl" scale="0.001 0.001 0.001"/>
     </geometry>
     <material name="silver"/>
@@ -40,5 +41,5 @@
     <origin xyz="0.075 0.3 0.36" rpy="0 0 0"/>
     <geometry>
-      <mesh filename="file://$(find Forkkun_description)/meshes/right_wheel_1.stl" scale="0.001 0.001 0.001"/>
+      <mesh filename="file://$(find forkkun_description)/meshes/right_wheel_1.stl" scale="0.001 0.001 0.001"/>
     </geometry>
   </collision>
@@ -53,5 +54,5 @@
     <origin xyz="0.075 -0.3 0.36" rpy="0 0 0"/>
     <geometry>
-      <mesh filename="file://$(find Forkkun_description)/meshes/left_wheel_1.stl" scale="0.001 0.001 0.001"/>
+      <mesh filename="file://$(find forkkun_description)/meshes/left_wheel_1.stl" scale="0.001 0.001 0.001"/>
     </geometry>
     <material name="silver"/>
@@ -60,5 +61,5 @@
     <origin xyz="0.075 -0.3 0.36" rpy="0 0 0"/>
     <geometry>
-      <mesh filename="file://$(find Forkkun_description)/meshes/left_wheel_1.stl" scale="0.001 0.001 0.001"/>
+      <mesh filename="file://$(find forkkun_description)/meshes/left_wheel_1.stl" scale="0.001 0.001 0.001"/>
     </geometry>
   </collision>
@@ -73,5 +74,5 @@
     <origin xyz="-1.35 0.35 0.47" rpy="0 0 0"/>
     <geometry>
-      <mesh filename="file://$(find Forkkun_description)/meshes/right_castor_1.stl" scale="0.001 0.001 0.001"/>
+      <mesh filename="file://$(find forkkun_description)/meshes/right_castor_1.stl" scale="0.001 0.001 0.001"/>
     </geometry>
     <material name="silver"/>
@@ -80,5 +81,5 @@
     <origin xyz="-1.35 0.35 0.47" rpy="0 0 0"/>
     <geometry>
-      <mesh filename="file://$(find Forkkun_description)/meshes/right_castor_1.stl" scale="0.001 0.001 0.001"/>
+      <mesh filename="file://$(find forkkun_description)/meshes/right_castor_1.stl" scale="0.001 0.001 0.001"/>
     </geometry>
   </collision>
@@ -93,5 +94,5 @@
     <origin xyz="-1.35 -0.35 0.47" rpy="0 0 0"/>
     <geometry>
-      <mesh filename="file://$(find Forkkun_description)/meshes/left_castor_1.stl" scale="0.001 0.001 0.001"/>
+      <mesh filename="file://$(find forkkun_description)/meshes/left_castor_1.stl" scale="0.001 0.001 0.001"/>
     </geometry>
     <material name="silver"/>
@@ -100,5 +101,5 @@
     <origin xyz="-1.35 -0.35 0.47" rpy="0 0 0"/>
     <geometry>
-      <mesh filename="file://$(find Forkkun_description)/meshes/left_castor_1.stl" scale="0.001 0.001 0.001"/>
+      <mesh filename="file://$(find forkkun_description)/meshes/left_castor_1.stl" scale="0.001 0.001 0.001"/>
     </geometry>
   </collision>
@@ -113,5 +114,5 @@
     <origin xyz="-0.45 -0.0 0.44" rpy="0 0 0"/>
     <geometry>
-      <mesh filename="file://$(find Forkkun_description)/meshes/carriage_1.stl" scale="0.001 0.001 0.001"/>
+      <mesh filename="file://$(find forkkun_description)/meshes/carriage_1.stl" scale="0.001 0.001 0.001"/>
     </geometry>
     <material name="silver"/>
@@ -120,5 +121,5 @@
     <origin xyz="-0.45 -0.0 0.44" rpy="0 0 0"/>
     <geometry>
-      <mesh filename="file://$(find Forkkun_description)/meshes/carriage_1.stl" scale="0.001 0.001 0.001"/>
+      <mesh filename="file://$(find forkkun_description)/meshes/carriage_1.stl" scale="0.001 0.001 0.001"/>
     </geometry>
   </collision>
