Commit message: Changed Carriage to be controlled by position instead of velocity

File: src/forkkun_description/urdf/Forkkun.ros2_control.xacro (robot description, xacro)
@@ -16,5 +16,5 @@
     </joint>
     <joint name="carriage">
-        <command_interface name="velocity"/>
+        <command_interface name="position"/>
         <state_interface name="position"/>
         <state_interface name="velocity"/>

File: src/forkkun_description/urdf/Forkkun.xacro (robot description, xacro)
@@ -150,9 +150,9 @@
 </joint>
 <joint name="carriage" type="prismatic">
-  <origin xyz="0.45 0.0 -0.44" rpy="0 0 0"/>
+  <origin xyz="0.45 0 0.44" rpy="0 0 0"/>
   <parent link="base_link"/>
   <child link="carriage_1"/>
   <axis xyz="0.0 0.0 1.0"/>
-  <limit upper="1.6" lower="0.0" effort="100" velocity="100"/>
+  <limit upper="1.6" lower="0.0" effort="2500" velocity="100"/>
 </joint>
 </robot>

Commit message: Revert "Changed Carriage to be controlled by position instead of velocity"
This reverts commit eaecaa4a2e8b15e357f8c67153900c82ab28f945.

File: src/forkkun_description/urdf/Forkkun.ros2_control.xacro (robot description, xacro)
@@ -16,5 +16,5 @@
     </joint>
     <joint name="carriage">
-        <command_interface name="position"/>
+        <command_interface name="velocity"/>
         <state_interface name="position"/>
         <state_interface name="velocity"/>

File: src/forkkun_description/urdf/Forkkun.xacro (robot description, xacro)
@@ -150,9 +150,9 @@
 </joint>
 <joint name="carriage" type="prismatic">
-  <origin xyz="0.45 0 0.44" rpy="0 0 0"/>
+  <origin xyz="0.45 0.0 -0.44" rpy="0 0 0"/>
   <parent link="base_link"/>
   <child link="carriage_1"/>
   <axis xyz="0.0 0.0 1.0"/>
-  <limit upper="1.6" lower="0.0" effort="2500" velocity="100"/>
+  <limit upper="1.6" lower="0.0" effort="100" velocity="100"/>
 </joint>
 </robot>
